File: MistFarm_PCB/MistFarm_PCB/3.3V.kicad_sch (KiCad schematic)
At the start: 9 parts, among them T1 Transformer_1P_1S, U1 L78L33_SOT89

Commit message: add sch
Parts:
- added 3.3v_ON: LED, LED_SMD:LED_0201_0603Metric, symbol Device:LED
- added R1: 1K, symbol Device:R
Connections:
- net 3.3V OUT: now also R1.2
- net GND: now also D2.2 (A), D4.2 (A), 3.3v_ON.1 (K); no longer D2.1 (K), D3.1 (K)
- net at C1.1, C2.1, D5.1 (K)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: now also D3.1 (K); no longer D3.2 (A)
- new net: 3.3v_ON.2 (A), R1.1
- new net: D2.1 (K), D3.2 (A), T1.3 (SA)
Other:
- moved on the sheet: D3

Commit message: sch and pcb modify
Parts:
- R16: renamed from R1; footprint (none) -> Resistor_SMD:R_0402_1005Metric
- renumbered 3.3v_ON to 3.3v_ON1, C1 to C19, C2 to C20, C3 to C21, D4 to D2, D5 to D3, D2 to D4, D3 to D5, U1 to U4
Connections:
- net 5A OUT: now reaches C19.1, C20.1, D3.1 (K), D5.1 (K), U4.3 (IN)
Changed lines of the file:
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@@
+	(wire
+		(pts
+			(xy 106.68 52.07) (xy 106.68 59.69)
+		)
+		(stroke
+			(width 0)
+			(type default)
+		)
+	)
 	(wire
 		(pts
@@
 		(property "Intersheetrefs" "${INTERSHEET_REFS}"
 			(at 171.7138 59.69 0)
+			(effects
+				(font
+					(size 1.27 1.27)
+				)
+				(justify left)
+				(hide yes)
+			)
+		)
+	)
+	(global_label "5A OUT"
+		(shape output)
+		(at 106.68 52.07 90)
+		(fields_autoplaced yes)
+		(effects
+			(font
+				(size 1.27 1.27)
+			)
+			(justify left)
+		)
+		(property "Intersheetrefs" "${INTERSHEET_REFS}"
+			(at 106.68 42.1905 90)
 			(effects
 				(font
@@
 		(dnp no)
 		(fields_autoplaced yes)
-		(property "Reference" "R1"
+		(property "Reference" "R16"
 			(at 152.4 52.0699 0)
 			(effects
@@
 			)
 		)
-		(property "Footprint" ""
+		(property "Footprint" "Resistor_SMD:R_0402_1005Metric"
 			(at 148.082 53.34 90)
 			(effects
@@
 			(project ""
 				(path "/341a7a15-82cf-4310-8068-7e972317a825/e87aa4b1-b142-4dda-94dc-9822a5c5d024"
-					(reference "R1")
+					(reference "R16")
 					(unit 1)
 				)
@@
 		(dnp no)
 		(fields_autoplaced yes)
-		(property "Reference" "C1"
+		(property "Reference" "C19"
 			(at 99.06 63.0681 0)
 			(effects
@@
 			(project ""
 				(path "/341a7a15-82cf-4310-8068-7e972317a825/e87aa4b1-b142-4dda-94dc-9822a5c5d024"
-					(reference "C1")
+					(reference "C19")
 					(unit 1)
 				)
@@
 		(dnp no)
 		(fields_autoplaced yes)
-		(property "Reference" "#PWR03"
+		(property "Reference" "#PWR025"
 			(at 149.86 31.75 0)
 			(effects
@@
 			(project "MistFarm_PCB"
 				(path "/341a7a15-82cf-4310-8068-7e972317a825/e87aa4b1-b142-4dda-94dc-9822a5c5d024"
-					(reference "#PWR03")
+					(reference "#PWR025")
 					(unit 1)
 				)
@@
 		(on_board yes)
 		(dnp no)
-		(property "Reference" "D4"
+		(property "Reference" "D2"
 			(at 67.564 64.262 90)
 			(effects
@@
 			(project "MistFarm_PCB"
 				(path "/341a7a15-82cf-4310-8068-7e972317a825/e87aa4b1-b142-4dda-94dc-9822a5c5d024"
-					(reference "D4")
+					(reference "D2")
 					(unit 1)
 				)
@@
 		(dnp no)
 		(fields_autoplaced yes)
-		(property "Reference" "D3"
+		(property "Reference" "D5"
 			(at 86.36 63.4999 90)
 			(effects
@@
 			(project "MistFarm_PCB"
 				(path "/341a7a15-82cf-4310-8068-7e972317a825/e87aa4b1-b142-4dda-94dc-9822a5c5d024"
-					(reference "D3")
+					(reference "D5")
 					(unit 1)
 				)
@@
 		(dnp no)
 		(fields_autoplaced yes)
-		(property "Reference" "C2"
+		(property "Reference" "C20"
 			(at 110.49 63.4999 0)
 			(effects
@@
 			(project ""
 				(path "/341a7a15-82cf-4310-8068-7e972317a825/e87aa4b1-b142-4dda-94dc-9822a5c5d024"
-					(reference "C2")
+					(reference "C20")
 					(unit 1)
 				)
@@
 		(dnp no)
 		(fields_autoplaced yes)
-		(property "Reference" "U1"
+		(property "Reference" "U4"
 			(at 124.46 53.34 0)
 			(effects
@@
 			(project ""
 				(path "/341a7a15-82cf-4310-8068-7e972317a825/e87aa4b1-b142-4dda-94dc-9822a5c5d024"
-					(reference "U1")
+					(reference "U4")
 					(unit 1)
 				)
@@
 		(dnp no)
 		(fields_autoplaced yes)
-		(property "Reference" "3.3v_ON"
+		(property "Reference" "3.3v_ON1"
 			(at 152.4 41.5924 90)
 			(effects
@@
 			(project ""
 				(path "/341a7a15-82cf-4310-8068-7e972317a825/e87aa4b1-b142-4dda-94dc-9822a5c5d024"
-					(reference "3.3v_ON")
+					(reference "3.3v_ON1")
 					(unit 1)
 				)
@@
 		(dnp no)
 		(fields_autoplaced yes)
-		(property "Reference" "D5"
+		(property "Reference" "D3"
 			(at 78.74 53.34 0)
 			(effects
@@
 			(project "MistFarm_PCB"
 				(path "/341a7a15-82cf-4310-8068-7e972317a825/e87aa4b1-b142-4dda-94dc-9822a5c5d024"
-					(reference "D5")
+					(reference "D3")
 					(unit 1)
 				)
@@
 		(dnp no)
 		(fields_autoplaced yes)
-		(property "Reference" "#PWR01"
+		(property "Reference" "#PWR024"
 			(at 115.57 77.47 0)
 			(effects
@@
 			(project ""
 				(path "/341a7a15-82cf-4310-8068-7e972317a825/e87aa4b1-b142-4dda-94dc-9822a5c5d024"
-					(reference "#PWR01")
+					(reference "#PWR024")
 					(unit 1)
 				)
@@
 		(on_board yes)
 		(dnp no)
-		(property "Reference" "D2"
+		(property "Reference" "D4"
 			(at 78.74 75.438 0)
 			(effects
@@
 			(project ""
 				(path "/341a7a15-82cf-4310-8068-7e972317a825/e87aa4b1-b142-4dda-94dc-9822a5c5d024"
-					(reference "D2")
+					(reference "D4")
 					(unit 1)
 				)
@@
 		(dnp no)
 		(fields_autoplaced yes)
-		(property "Reference" "C3"
+		(property "Reference" "C21"
 			(at 144.78 63.4999 0)
 			(effects
@@
 			(project "MistFarm_PCB"
 				(path "/341a7a15-82cf-4310-8068-7e972317a825/e87aa4b1-b142-4dda-94dc-9822a5c5d024"
-					(reference "C3")
-					(unit 1)
-				)
+					(reference "C21")
+					(unit 1)
+				)

Commit message: PCB update
Parts:
- 3.3v_ON1: value LED -> LTST-C190GKT
Changed lines of the file:
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@@
 			)
 		)
-		(property "Value" "LED"
+		(property "Value" "LTST-C190GKT"
 			(at 152.4 44.1324 90)
 			(effects

Commit message: PCB update
Parts:
- C19: footprint (none) -> Capacitor_SMD:C_1210_3225Metric
- C20, C21: footprint (none) -> Capacitor_SMD:C_0603_1608Metric
Changed lines of the file:
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@@
 			)
 		)
-		(property "Footprint" ""
+		(property "Footprint" "Capacitor_SMD:C_1210_3225Metric"
 			(at 96.52 64.77 0)
 			(effects
@@
 			)
 		)
-		(property "Footprint" ""
+		(property "Footprint" "Capacitor_SMD:C_0603_1608Metric"
 			(at 107.6452 68.58 0)
 			(effects
@@
 			)
 		)
-		(property "Footprint" ""
+		(property "Footprint" "Capacitor_SMD:C_0603_1608Metric"
 			(at 141.9352 68.58 0)
 			(effects

Commit message: PCB end
Parts:
- C14: renamed from C19; footprint Capacitor_SMD:C_1210_3225Metric -> footprints:CAPMP7.6X4.3_4.3N_KEM-L
- C16: renamed from C21; value 100nF -> 0.1uF
- renumbered C20 to C15, R16 to R13
Changed lines of the file:
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@@
 		(dnp no)
 		(fields_autoplaced yes)
-		(property "Reference" "R16"
+		(property "Reference" "R13"
 			(at 152.4 52.0699 0)
 			(effects
@@
 			(project ""
 				(path "/341a7a15-82cf-4310-8068-7e972317a825/e87aa4b1-b142-4dda-94dc-9822a5c5d024"
-					(reference "R16")
+					(reference "R13")
 					(unit 1)
 				)
@@
 		(dnp no)
 		(fields_autoplaced yes)
-		(property "Reference" "C19"
+		(property "Reference" "C14"
 			(at 99.06 63.0681 0)
 			(effects
@@
 			)
 		)
-		(property "Footprint" "Capacitor_SMD:C_1210_3225Metric"
+		(property "Footprint" "footprints:CAPMP7.6X4.3_4.3N_KEM-L"
 			(at 96.52 64.77 0)
 			(effects
@@
 			)
 		)
-		(property "Description" "Polarized capacitor, small US symbol"
+		(property "Description" "Polarized capacitor, small US symbol, T495X477K010ATE100"
 			(at 96.52 64.77 0)
 			(effects
@@
 			(project ""
 				(path "/341a7a15-82cf-4310-8068-7e972317a825/e87aa4b1-b142-4dda-94dc-9822a5c5d024"
-					(reference "C19")
+					(reference "C14")
 					(unit 1)
 				)
@@
 		(dnp no)
 		(fields_autoplaced yes)
-		(property "Reference" "#PWR025"
+		(property "Reference" "#PWR021"
 			(at 149.86 31.75 0)
 			(effects
@@
 			(project "MistFarm_PCB"
 				(path "/341a7a15-82cf-4310-8068-7e972317a825/e87aa4b1-b142-4dda-94dc-9822a5c5d024"
-					(reference "#PWR025")
+					(reference "#PWR021")
 					(unit 1)
 				)
@@
 		(dnp no)
 		(fields_autoplaced yes)
-		(property "Reference" "C20"
+		(property "Reference" "C15"
 			(at 110.49 63.4999 0)
 			(effects
@@
 			(project ""
 				(path "/341a7a15-82cf-4310-8068-7e972317a825/e87aa4b1-b142-4dda-94dc-9822a5c5d024"
-					(reference "C20")
+					(reference "C15")
 					(unit 1)
 				)
@@
 		(dnp no)
 		(fields_autoplaced yes)
-		(property "Reference" "#PWR024"
+		(property "Reference" "#PWR020"
 			(at 115.57 77.47 0)
 			(effects
@@
 			(project ""
 				(path "/341a7a15-82cf-4310-8068-7e972317a825/e87aa4b1-b142-4dda-94dc-9822a5c5d024"
-					(reference "#PWR024")
+					(reference "#PWR020")
 					(unit 1)
 				)
@@
 		(dnp no)
 		(fields_autoplaced yes)
-		(property "Reference" "C21"
+		(property "Reference" "C16"
 			(at 144.78 63.4999 0)
 			(effects
@@
 			)
 		)
-		(property "Value" "100nF"
+		(property "Value" "0.1uF"
 			(at 144.78 66.0399 0)
 			(effects
@@
 			(project "MistFarm_PCB"
 				(path "/341a7a15-82cf-4310-8068-7e972317a825/e87aa4b1-b142-4dda-94dc-9822a5c5d024"
-					(reference "C21")
-					(unit 1)
-				)
+					(reference "C16")
+					(unit 1)
+				)

Commit message: PCB real end
Parts:
- added C23: 470uF, footprints:CAPMP7.6X4.3_4.3N_KEM-L, symbol Device:C_Polarized_Small_US
- added C24, C25: 0.1uF, Capacitor_SMD:C_0603_1608Metric, symbol Device:C
- added Q2: UMH3N, Package_TO_SOT_SMD:SOT-363_SC-70-6, symbol Transistor_BJT:UMH3N
- added U7, U8: L78L33_SOT89, Package_TO_SOT_SMD:SOT-89-3, symbol Regulator_Linear:L78L33_SOT89
Connections:
- net 5A OUT: now also C23.1, U7.3 (IN), U8.3 (IN)
- net GND: now also C23.2, C24.2, C25.2, U7.2 (GND), U8.2 (GND)
- new net: Q2.6 (C1), U8.1 (OUT)
- new net: Q2.3 (C2), U7.1 (OUT)
- new net Moter_A: Q2.1 (E1)
- new net Moter_A_triger: C24.1, Q2.2 (B1)
- new net Moter_B: Q2.4 (E2)
- new net Moter_B_triger: C25.1, Q2.5 (B2)
Other:
- moved on the sheet: C15
