File: MistFarm_PCB/MistFarm_PCB/MistFarm_PCB.kicad_pcb (KiCad board)
At the start: 2 copper layers, 44 parts, among them J5 GRPB052VWVN-RC, J6 OLED, Q3 UMH3N, U2 ESP32-WROOM-32E, U6 CP2104, U9 USBLC6-2P6

Commit message: sch and pcb modify
Parts:
- added 3.3v_ON1: LED, LED_SMD:LED_0201_0603Metric, F.Cu at (44.0, 66.1)
- added D2: 1N4007, 1N4007FLTR:SODFL3618X110N, F.Cu at (60.1, 77.8)
- added D3: 1N4007, 1N4007FLTR:SODFL3618X110N, F.Cu at (56.2, 81.6)
- added D4: 1N4007, 1N4007FLTR:SODFL3618X110N, F.Cu at (56.1, 73.7)
- added D5: 1N4007, 1N4007FLTR:SODFL3618X110N, F.Cu at (52.1, 77.8)
- added D6: 1N4007, 1N4007FLTR:SODFL3618X110N, F.Cu at (177.2, 76.6)
- added D7: 1N4007, 1N4007FLTR:SODFL3618X110N, F.Cu at (177.2, 80.0)
- added NTCG103JX103DT1S1: 10K, Resistor_SMD:R_0603_1608Metric, F.Cu at (170.5, 69.2)
- added R16: 1K, Resistor_SMD:R_0603_1608Metric, F.Cu at (45.2, 66.9)
- added R17: 75, Resistor_SMD:R_0603_1608Metric, F.Cu at (185.7, 77.0)
- added U4: L78L33_SOT89, Package_TO_SOT_SMD:SOT-89-3, F.Cu at (48.0, 73.3)
- added U5: SHT45-AD1B-R3, SHT45-AD1B-R3:SHT4x_SEN, F.Cu at (176.4, 83.3)
- J2: renamed from J6; value OLED -> I2C
- R11: renamed from R25; footprint Resistor_SMD:R_0402_1005Metric -> Resistor_SMD:R_0603_1608Metric
- R12: renamed from R26; footprint Resistor_SMD:R_0402_1005Metric -> Resistor_SMD:R_0603_1608Metric
- R14: renamed from R28; footprint Resistor_SMD:R_0402_1005Metric -> Resistor_SMD:R_0603_1608Metric
- R15: renamed from R29; footprint Resistor_SMD:R_0402_1005Metric -> Resistor_SMD:R_0603_1608Metric
- R5: renamed from R31; footprint Resistor_SMD:R_0402_1005Metric -> Resistor_SMD:R_0603_1608Metric
- moved C9 86.7 mm to (78.7, 112.1), turned to -90 degrees
- moved C10 84.3 mm to (76.5, 112.1), turned to -90 degrees
- moved C11 75.2 mm to (83.2, 102.3)
- moved C12 75.2 mm to (83.2, 104.8)
- moved R4 70.0 mm to (89.0, 34.7), turned to 90 degrees
- moved D1 69.6 mm to (38.8, 75.3), turned to 0 degrees
- moved R3 67.2 mm to (87.2, 34.7), turned to 90 degrees
- moved R7 66.2 mm to (79.5, 105.7), turned to 90 degrees
- moved R2 64.5 mm to (85.4, 34.7), turned to 90 degrees
- moved R10 62.9 mm to (77.3, 105.7), turned to 90 degrees
- moved R1 61.9 mm to (83.7, 34.7), turned to 90 degrees
- moved J2 57.3 mm to (81.0, 109.5)
- moved C13 56.5 mm to (75.1, 61.2), turned to 180 degrees
- moved C15 55.8 mm to (75.0, 57.4), turned to 180 degrees
- moved F1 54.2 mm to (74.9, 53.6)
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- renumbered C38 to C1, C24 to C10, C25 to C11, C26 to C12, C33 to C13, C34 to C14, C12 to C15, C39 to C16, C40 to C17, C41 to C18, C32 to C2, C11 to C3, C20 to C4, C21 to C5, C22 to C6, C36 to C7, C7 to C8, C23 to C9, F2 to F1, FL2 to FL1, J5 to J1, Q3 to Q1, R16 to R1, R24 to R10, R27 to R13, R17 to R2, R18 to R3, R19 to R4, R20 to R6, R23 to R7, R34 to R8, R35 to R9, S2 to S1, U2 to U1, U6 to U2, U9 to U3, UART2 to UART1
Connections:
- net INPUT AC1 renamed /3.3V generator/Transformer_input_A
- net OUTPUT AC1 renamed /HIGH_AC_Switching/OUTPUT_AC1
- FL1 pad 2: Net-(FL2-Pad2) -> 5A OUT
- U1 pad 10: unconnected-(U2-IO25-Pad10) -> /ESP32 WROOM 32E/Temp_Sensor
- UART1 pad A1_B12: (no net) -> GND
- UART1 pad A4_B9: (no net) -> 5A OUT
- UART1 pad B1_A12: (no net) -> GND
- UART1 pad B4_A9: (no net) -> 5A OUT
Routing:
- net /3.3V generator/Transformer_input_A: track 21.3 -> 163.7 mm
- net /ESP32 WROOM 32E/I2C_SCL: track 0.00 -> 121.6 mm, vias 0 -> 1
- net /ESP32 WROOM 32E/I2C_SDL: track 0.00 -> 117.3 mm, vias 0 -> 1
- net /ESP32 WROOM 32E/EN: track 0.00 -> 91.7 mm, vias 0 -> 2
- net 5A OUT: track 0.00 -> 68.8 mm, vias 0 -> 2
- net GND: track 0.00 -> 66.0 mm, vias 0 -> 20
- net /ESP32 WROOM 32E/JTAG_MTMS: track 0.00 -> 64.2 mm, vias 0 -> 2
- net /ESP32 WROOM 32E/JTAG_MTDI: track 0.00 -> 59.8 mm, vias 0 -> 2
- net /ESP32 WROOM 32E/JTAG_MTCK: track 0.00 -> 54.9 mm, vias 0 -> 2
- net /ESP32 WROOM 32E/AC_TRIAC_Switching: track 0.00 -> 50.1 mm, vias 0 -> 2
- net /ESP32 WROOM 32E/JTAG_MTDO: track 0.00 -> 44.5 mm, vias 0 -> 2
- net 3.3V OUT: track 0.00 -> 41.5 mm, vias 0 -> 7
- net Net-(D4-K): track 0.00 -> 22.5 mm, vias 0 -> 2
- net /ESP32 WROOM 32E/RTS: track 0.00 -> 20.5 mm, vias 0 -> 3
- net Net-(U2-REGIN): track 0.00 -> 18.4 mm, vias 0 -> 4
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- added copper zone on In1.Cu, net 3.3V OUT
- added copper zone on B.Cu, net GND
- added copper zone on F.Cu, net GND
- added copper zone on In2.Cu, net GND
Other:
- board outline added: 98.4 x 95.2 mm
- copper layers 2 -> 4

Commit message: PCB update
Parts:
- added J3: 61300511121, 61300511121:61300511121, F.Cu at (89.1, 90.0)
- added J4: 61300511121, 61300511121:61300511121, F.Cu at (112.8, 24.0)
- NTCG103JX103DT1S1, R11, R12, R14, R15, R16, R17, R5: footprint Resistor_SMD:R_0603_1608Metric -> Resistor_SMD:R_0402_1005Metric
- moved R17 86.7 mm to (111.0, 33.0), turned to 180 degrees
- moved D7 86.2 mm to (108.4, 28.0)
- moved D6 79.5 mm to (114.4, 28.0)
- moved U5 77.4 mm to (117.9, 32.6)
- moved NTCG103JX103DT1S1 72.2 mm to (108.0, 33.1)
- moved R16 1.14 mm to (45.2, 65.8), turned to 90 degrees
- moved C3 0.38 mm to (90.3, 21.4)
- moved C4 0.38 mm to (90.3, 23.7)
- moved C5 0.38 mm to (90.3, 25.8)
- moved C6 0.38 mm to (90.3, 28.0)
Connections:
- UART1 pad SH1: (no net) -> GND
- UART1 pad SH2: (no net) -> GND
- UART1 pad SH3: (no net) -> GND
- UART1 pad SH4: (no net) -> GND
Routing:
- net /ESP32 WROOM 32E/Temp_Sensor: track 0.00 -> 125.2 mm, vias 0 -> 2
- net GND: track 66.0 -> 107.0 mm, vias 20 -> 23
- net /ESP32 WROOM 32E/I2C_SCL: track 121.6 -> 159.9 mm, vias 1 -> 2
- net /ESP32 WROOM 32E/I2C_SDL: track 117.3 -> 155.2 mm, vias 1 -> 2
- net 3.3V OUT: track 41.5 -> 66.1 mm
- net Net-(C3-Pad1): track 16.0 -> 27.4 mm
Other:
- board size 98.4 x 95.2 mm -> 103.4 x 95.2 mm
- board text added: "3.3v"
- board text added: "GND"
- board text added: "J3"
- board text added: "SCL"
- board text added: "SDL"
- board text added: "Temp_Sensor"

Commit message: PCB update
Other:
- outline, holes or cut-outs redrawn
- board text removed: "J3"
Changed lines of the file:
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@@
 				(thickness 0.035)
 			)
-			(layer "dielectric 1"
+			(layer "dielectric 4"
 				(type "prepreg")
 				(thickness 0.1)
@@
 				(thickness 0.035)
 			)
-			(layer "dielectric 2"
+			(layer "dielectric 5"
 				(type "core")
 				(thickness 1.24)
@@
 				(thickness 0.035)
 			)
-			(layer "dielectric 3"
+			(layer "dielectric 6"
 				(type "prepreg")
 				(thickness 0.1)
@@
 			(outputformat 1)
 			(mirror no)
-			(drillshape 1)
+			(drillshape 0)
 			(scaleselection 1)
 			(outputdirectory "")
@@
 		(net 15)
 	)
+	(gr_line
+		(start 91.840136 55.199863)
+		(end 91.84 114.35)
+		(stroke
+			(width 0.05)
+			(type default)
+		)
+		(layer "Edge.Cuts")
+	)
+	(gr_arc
+		(start 90.030137 53.389863)
+		(mid 91.31 53.92)
+		(end 91.840137 55.199863)
+		(stroke
+			(width 0.05)
+			(type default)
+		)
+		(layer "Edge.Cuts")
+	)
+	(gr_line
+		(start 91.84 19.11)
+		(end 17.48 19.11)
+		(stroke
+			(width 0.05)
+			(type default)
+		)
+		(layer "Edge.Cuts")
+	)
+	(gr_arc
+		(start 88.873033 43.42)
+		(mid 89.220484 42.645488)
+		(end 90.03 42.39)
+		(stroke
+			(width 0.05)
+			(type default)
+		)
+		(layer "Edge.Cuts")
+	)
+	(gr_line
+		(start 91.84 19.11)
+		(end 91.84 40.58)
+		(stroke
+			(width 0.05)
+			(type default)
+		)
+		(layer "Edge.Cuts")
+	)
+	(gr_line
+		(start 17.48 19.11)
+		(end 17.48 114.35)
+		(stroke
+			(width 0.05)
+			(type default)
+		)
+		(layer "Edge.Cuts")
+	)
+	(gr_line
+		(start 17.48 114.35)
+		(end 91.84 114.35)
+		(stroke
+			(width 0.05)
+			(type default)
+		)
+		(layer "Edge.Cuts")
+	)
 	(gr_rect
 		(start 104.02 20.3)
@@
 		(layer "Edge.Cuts")
 	)
-	(gr_rect
-		(start 17.48 19.11)
-		(end 91.84 114.35)
+	(gr_line
+		(start 88.873033 43.42)
+		(end 88.87317 52.3599)
 		(stroke
 			(width 0.05)
 			(type default)
 		)
-		(fill no)
 		(layer "Edge.Cuts")
 	)
-	(gr_text "J3"
-		(at 157.97 113.18 180)
-		(layer "F.SilkS")
-		(effects
-			(font
-				(size 0.8 0.8)
-				(thickness 0.15)
-			)
+	(gr_arc
+		(start 90.030137 53.389863)
+		(mid 89.220621 53.134375)
+		(end 88.87317 52.359863)
+		(stroke
+			(width 0.05)
+			(type default)
 		)
+		(layer "Edge.Cuts")
+	)
+	(gr_arc
+		(start 91.84 40.58)
+		(mid 91.309863 41.859863)
+		(end 90.03 42.39)
+		(stroke
+			(width 0.05)
+			(type default)
+		)
+		(layer "Edge.Cuts")
 	)
 	(gr_text "SDL"

Commit message: PCB update
Parts:
- added C19: 470uF, MAL214097013E3:MAL214097013E3, F.Cu at (72.5, 79.9)
- added C20: 300nF, Capacitor_SMD:C_0603_1608Metric, F.Cu at (46.4, 88.2)
- added C21: 100nF, Capacitor_SMD:C_0603_1608Metric, F.Cu at (53.9, 64.5)
Routing:
- net 5A OUT: track 68.8 -> 117.7 mm
- net 3.3V OUT: track 66.1 -> 68.1 mm
- net GND: track 107.0 -> 109.0 mm

Commit message: PCB end
Parts:
- moved U5 137.7 mm to (19.2, 128.6), turned to -90 degrees
- moved D6 132.7 mm to (23.8, 125.0), turned to -90 degrees
- moved J4 130.8 mm to (27.8, 123.4), turned to -90 degrees
- moved R17 127.8 mm to (18.8, 121.6), turned to 90 degrees
- moved D7 124.3 mm to (23.8, 119.1), turned to -90 degrees
- moved NTCG103JX103DT1S1 123.7 mm to (18.7, 118.7), turned to 90 degrees
Other:
- board size 103.4 x 95.2 mm -> 74.4 x 112.4 mm

Commit message: PCB end
Parts:
- removed C17: 0.1uF, Capacitor_SMD:C_0603_1608Metric
- removed C18: 4.7uF, Capacitor_SMD:C_0603_1608Metric
- removed C19: 470uF, MAL214097013E3:MAL214097013E3
- removed C20: 300nF, Capacitor_SMD:C_0603_1608Metric
- removed C21: 100nF, Capacitor_SMD:C_0603_1608Metric
- removed F1: 0603L100SLYR, Resistor_SMD:R_0603_1608Metric
- removed FL1: BLM21PG221SN1D, BLM21PG221SN1D:BEADC2012X105N
- removed NTCG103JX103DT1S1: 10K, Resistor_SMD:R_0402_1005Metric
- removed the R13 at (79.2, 58.1)
- removed R15: 5.1K, Resistor_SMD:R_0402_1005Metric
- removed R17: 75, Resistor_SMD:R_0402_1005Metric
- removed UART1: 12402012E212A, 12402012E212A:AMPHENOL_12402012E212A
- added J1: 61300511121, 61300511121:61300511121, F.Cu at (27.8, 123.5)
- added Temp_sensor: 10K, Resistor_SMD:R_0402_1005Metric, F.Cu at (18.8, 118.7)
- 3.3v_ON1: value LED -> LTST-C190GKT
- C13: value 0.1uF -> 10uF; footprint Capacitor_SMD:C_0603_1608Metric -> Capacitor_SMD:C_0805_2012Metric
- C14: value 22uF -> 470uF; footprint Capacitor_SMD:C_0805_2012Metric -> footprints:CAPMP7.6X4.3_4.3N_KEM-L
- C15: value 4.7uF -> 300nF
- C16: value 22uF -> 100nF; footprint Capacitor_SMD:C_0805_2012Metric -> Capacitor_SMD:C_0603_1608Metric
- J3: renamed from J2; value I2C -> HTSW-104-20-TM-S
- J4: value 61300511121 -> 12402012E212A; footprint 61300511121:61300511121 -> 12402012E212A:AMPHENOL_12402012E212A
- R11, R12: value 22R -> 5.1K
- R14: value 5.1K -> 75
- U5: footprint SHT45-AD1B-R3:SHT4x_SEN -> SHT45_AD1B_R3:SHT4x_SEN
- moved J4 96.4 mm to (87.8, 47.9), turned to 90 degrees
- moved R14 86.6 mm to (18.8, 121.6), turned to 90 degrees
- moved C16 29.5 mm to (46.9, 68.4), turned to 0 degrees
- moved C15 26.7 mm to (69.7, 83.5), turned to 0 degrees
- moved C13 21.8 mm to (53.4, 63.5), turned to 0 degrees
- moved C14 17.6 mm to (69.7, 79.9)
- moved R12 16.6 mm to (79.9, 53.3)
- moved R11 16.4 mm to (79.9, 51.3)
- moved R8 9.22 mm to (65.4, 50.1), turned to 0 degrees
- moved R9 5.93 mm to (65.4, 51.8), turned to 0 degrees
- moved U2 0.99 mm to (70.9, 47.6), turned to 0 degrees
- moved Q1 0.87 mm to (69.6, 53.8), turned to 0 degrees
- moved C7 0.66 mm to (53.3, 66.5)
- moved C8 0.64 mm to (53.4, 68.7)
- moved U3 0.29 mm to (77.2, 47.9)
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- renumbered J1 to J2, J3 to J5, R16 to R13
Connections:
- net /ESP32 WROOM 32E/SPI_Reset renamed /ESP32 WROOM 32E/GPS_TX2
- C14 pad 1: GND -> 5A OUT
- C14 pad 2: 3.3V OUT -> GND
- C15 pad 1: Net-(U2-REGIN) -> 5A OUT
- C16 pad 1: Net-(U2-REGIN) -> 3.3V OUT
- R11 pad 1: /ESP32 WROOM 32E/TX -> GND
- R11 pad 2: Net-(U2-RXD) -> Net-(J4-CC2)
- R12 pad 1: /ESP32 WROOM 32E/RX -> GND
- R12 pad 2: Net-(U2-TXD) -> Net-(J4-CC1)
- R14 pad 2: Net-(UART1-CC2) -> /ESP32 WROOM 32E/Temp_Sensor
- U1 pad 12: unconnected-(U1-IO27-Pad12) -> /ESP32 WROOM 32E/AC_TRIAC_Switching
- U1 pad 28: /ESP32 WROOM 32E/AC_TRIAC_Switching -> /ESP32 WROOM 32E/GPS_RX2
- U2 pad 16: Net-(U2-VPP) -> unconnected-(U2-VPP-Pad16)
- U2 pad 20: Net-(U2-RXD) -> /ESP32 WROOM 32E/TX
- U2 pad 21: Net-(U2-TXD) -> /ESP32 WROOM 32E/RX
- U2 pad 7: Net-(U2-REGIN) -> 3.3V OUT
- U2 pad 8: Net-(U2-REGIN) -> 5A OUT
- U2 pad 9: Net-(U2-~{RST}) -> unconnected-(U2-~{RST}-Pad9)
- U3 pad 1: Net-(U3-I/O1-Pad1) -> Net-(J4-D--PadA7)
- U3 pad 3: Net-(U3-I/O2-Pad3) -> Net-(J4-D+-PadA6)
- U3 pad 4: Net-(U2-D-) -> Net-(U2-D+)
- U3 pad 5: Net-(U2-REGIN) -> 5A OUT
- U3 pad 6: Net-(U2-D+) -> Net-(U2-D-)
Routing:
- net /ESP32 WROOM 32E/AC_TRIAC_Switching: track 50.1 -> 30.3 mm
- net 5A OUT: track 117.7 -> 137.1 mm, vias 2 -> 4
- net Net-(U2-REGIN): track 18.4 -> 0.00 mm, vias 4 -> 0
- net Net-(UART1-CC2): track 15.8 -> 0.00 mm, vias 2 -> 0
- net Net-(U2-~{RST}): track 14.7 -> 0.00 mm, vias 2 -> 0
- net Net-(UART1-CC1): track 13.6 -> 0.00 mm
- net /ESP32 WROOM 32E/TX: track 4.78 -> 15.6 mm
- net /ESP32 WROOM 32E/RX: track 4.76 -> 15.2 mm
- net Net-(U3-I/O2-Pad3): track 8.16 -> 0.00 mm
- net Net-(J4-D+-PadA6): track 0.00 -> 7.74 mm
- net GND: track 109.0 -> 101.5 mm, vias 23 -> 15
- net Net-(U3-I/O1-Pad1): track 7.49 -> 0.00 mm, vias 3 -> 0
- net Net-(J4-CC2): track 0.00 -> 7.49 mm, vias 0 -> 2
- net Net-(J4-D--PadA7): track 0.00 -> 6.86 mm
- net /ESP32 WROOM 32E/DTR: track 11.6 -> 18.2 mm, vias 0 -> 2
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
Commit message: PCB real end
Parts:
- removed C3, C4, C5, C6: PESD0402-140, PESD0402-140:RESC1005X35N
- removed R1, R2, R3, R4: 100R, Resistor_SMD:R_0603_1608Metric
- added C17: 4.7uF, Capacitor_SMD:C_0603_1608Metric, F.Cu at (87.1, 79.5)
- added C18: 0.1uF, Capacitor_SMD:C_0603_1608Metric, F.Cu at (87.1, 82.0)
- added C19: 4.7uF, Capacitor_SMD:C_0603_1608Metric, F.Cu at (84.5, 37.0)
- added C20: 0.1uF, Capacitor_SMD:C_0603_1608Metric, F.Cu at (84.5, 38.9)
- added C21: 1uF, Capacitor_SMD:C_0603_1608Metric, F.Cu at (84.5, 40.8)
- added C22: 22uF, Capacitor_SMD:C_0805_2012Metric, F.Cu at (80.5, 82.5)
- added C23: 470uF, footprints:CAPMP7.6X4.3_4.3N_KEM-L, F.Cu at (67.4, 90.5)
- added C24: 0.1uF, Capacitor_SMD:C_0603_1608Metric, F.Cu at (79.6, 36.6)
- added C25: 0.1uF, Capacitor_SMD:C_0603_1608Metric, F.Cu at (79.6, 34.1)
- added J6: 6130XX11121_61300811121, 61300811121:61300811121, F.Cu at (79.2, 111.0)
- added Q2: UMH3N, Package_TO_SOT_SMD:SOT-363_SC-70-6, F.Cu at (83.6, 30.2)
- added U6: L86-M33, L86-M33:XCVR_L86-M33, F.Cu at (74.0, 70.5)
- added U7: L78L33_SOT89, Package_TO_SOT_SMD:SOT-89-3, F.Cu at (65.2, 84.6)
- added U8: L78L33_SOT89, Package_TO_SOT_SMD:SOT-89-3, F.Cu at (71.1, 84.5)
- C16: value 100nF -> 0.1uF
- J2: value GRPB052VWVN-RC -> 6130XX11121_61300811121; footprint Varistor:SULLINS_GRPB052VWVN-RC -> 61300811121:61300811121
- J3: value HTSW-104-20-TM-S -> 6130XX11121_61300811121; footprint HTSW-104-20-TM-S:SAMTEC_HTSW-104-20-TM-S -> 61300811121:61300811121
- moved J3 79.3 mm to (88.8, 30.5), turned to 90 degrees
- moved J2 43.5 mm to (88.8, 67.9), turned to 90 degrees
- moved C10 27.0 mm to (82.8, 85.8), turned to 180 degrees
- moved C9 25.0 mm to (82.8, 87.5), turned to 180 degrees
- moved R10 20.2 mm to (80.0, 85.7), turned to 180 degrees
- moved C14 19.1 mm to (66.9, 98.7)
- moved R7 18.2 mm to (80.0, 87.5), turned to 180 degrees
- moved C15 11.4 mm to (66.6, 94.5)
- moved J1 4.18 mm to (28.4, 127.6)
- moved D6 4.18 mm to (24.4, 129.2)
- moved D7 4.18 mm to (24.4, 123.3)
- moved R14 4.18 mm to (19.4, 125.7)
- moved Temp_NTC 4.18 mm to (19.4, 122.8)
- moved U5 4.18 mm to (19.8, 132.7)
- renumbered Temp_sensor to Temp_NTC
Connections:
- C11 pad 1: 3.3V OUT -> GND
- C11 pad 2: GND -> 3.3V OUT
- C12 pad 1: 3.3V OUT -> GND
- C12 pad 2: GND -> 3.3V OUT
- J2 pad 2: Net-(C3-Pad1) -> GND
- J2 pad 3: GND -> /ESP32 WROOM 32E/GPIO14
- J2 pad 4: Net-(C4-Pad1) -> /ESP32 WROOM 32E/GPIO13
- J2 pad 5: GND -> /ESP32 WROOM 32E/GPIO12
- J2 pad 6: Net-(C5-Pad1) -> /ESP32 WROOM 32E/GPIO5
- J2 pad 7: unconnected-(J2-Pad7) -> /ESP32 WROOM 32E/GPIO4
- J2 pad 8: Net-(C6-Pad1) -> /ESP32 WROOM 32E/GPIO2
- U1 pad 11: /ESP32 WROOM 32E/SPI_DIO0(IRQ) -> /ESP32 WROOM 32E/GPIO26
- U1 pad 13: /ESP32 WROOM 32E/JTAG_MTMS -> /ESP32 WROOM 32E/GPIO14
- U1 pad 14: /ESP32 WROOM 32E/JTAG_MTDI -> /ESP32 WROOM 32E/GPIO12
- U1 pad 16: /ESP32 WROOM 32E/JTAG_MTCK -> /ESP32 WROOM 32E/GPIO13
- U1 pad 23: /ESP32 WROOM 32E/JTAG_MTDO -> /ESP32 WROOM 32E/GPIO15
- U1 pad 24: unconnected-(U1-IO2-Pad24) -> /ESP32 WROOM 32E/GPIO2
- U1 pad 26: unconnected-(U1-IO4-Pad26) -> /ESP32 WROOM 32E/GPIO4
- U1 pad 27: /ESP32 WROOM 32E/GPS_TX2 -> /ESP32 WROOM 32E/GPIO16
- U1 pad 28: /ESP32 WROOM 32E/GPS_RX2 -> /ESP32 WROOM 32E/GPIO17
- U1 pad 29: /ESP32 WROOM 32E/SPI_SCK -> /ESP32 WROOM 32E/GPIO5
- U1 pad 30: /ESP32 WROOM 32E/SPI_NSS(CS) -> /3.3V generator/Moter_B_triger
- U1 pad 31: /ESP32 WROOM 32E/SPI_MISO -> /3.3V generator/Moter_A_triger
- U1 pad 37: /ESP32 WROOM 32E/SPI_MOSI -> /ESP32 WROOM 32E/GPIO23
- U1 pad 6: unconnected-(U1-IO34-Pad6) -> /ESP32 WROOM 32E/GPIO34
- U1 pad 7: unconnected-(U1-IO35-Pad7) -> /ESP32 WROOM 32E/GPIO35
- U1 pad 8: unconnected-(U1-IO32-Pad8) -> /ESP32 WROOM 32E/GPIO32
- U1 pad 9: unconnected-(U1-IO33-Pad9) -> /ESP32 WROOM 32E/GPIO33
Routing:
- net 3.3V OUT: track 62.0 -> 270.1 mm, vias 7 -> 12
- net /ESP32 WROOM 32E/GPIO23: track 0.00 -> 118.2 mm, vias 0 -> 3
- net /ESP32 WROOM 32E/GPIO26: track 0.00 -> 98.8 mm, vias 0 -> 4
- net /ESP32 WROOM 32E/GPIO32: track 0.00 -> 97.6 mm, vias 0 -> 4
- net /ESP32 WROOM 32E/GPIO34: track 0.00 -> 88.0 mm, vias 0 -> 4
- net GND: track 101.5 -> 188.8 mm, vias 15 -> 23
- net /ESP32 WROOM 32E/GPIO33: track 0.00 -> 87.2 mm, vias 0 -> 4
- net /ESP32 WROOM 32E/GPIO35: track 0.00 -> 83.8 mm, vias 0 -> 4
- net Net-(Q2B-C2): track 0.00 -> 66.8 mm, vias 0 -> 2
- net /ESP32 WROOM 32E/GPIO15: track 0.00 -> 65.1 mm, vias 0 -> 1
- net /ESP32 WROOM 32E/GPIO16: track 0.00 -> 64.8 mm, vias 0 -> 2
- net Net-(Q2A-C1): track 0.00 -> 64.3 mm, vias 0 -> 2
- net /ESP32 WROOM 32E/JTAG_MTMS: track 64.2 -> 0.00 mm, vias 2 -> 0
- net /ESP32 WROOM 32E/GPIO12: track 0.00 -> 63.5 mm, vias 0 -> 2
- net /ESP32 WROOM 32E/GPIO17: track 0.00 -> 60.7 mm, vias 0 -> 2
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- removed copper zone on In1.Cu, net 3.3V OUT
- removed copper zone on In2.Cu, net GND
Other:
- board size 74.4 x 112.4 mm -> 74.4 x 116.6 mm
- copper layers 4 -> 2
- board text added: "12"
- board text added: "13"
- board text added: "14"
- board text added: "15"
- board text added: "16"
- board text added: "17"
- board text added: "18"
- board text added: "19"
- board text added: "2"
- board text added: "220V input"
- board text added: "23"
- board text added: "26"
- board text added: "32"
- board text added: "33"
- board text added: "34"
- board text added: "35"
- board text added: "4"
- board text added: "5"
- board text added: "Transformer"
